File: elec/src/lv2842xlvddcr/elec/layout/default/lv2842xlvddcr.kicad_pcb (KiCad board)
At the start: 2 copper layers, 225.7 x 100.8 mm, 0 parts

Commit message: layout progress
Parts:
- added C1: 10V 10uF X5R ±10% 0603 Multilayer Ceramic Capacitors MLCC -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, lib:C0603, F.Cu at (165.6, 89.4)
- added C2: 25V 10uF X5R ±10% 0805 Multilayer Ceramic Capacitors MLCC -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, lib:C0805, F.Cu at (161.9, 89.5)
- added C3: 16V 100nF X7R ±10% 0402 Multilayer Ceramic Capacitors MLCC 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, lib:C0402, F.Cu at (165.4, 94.2)
- added DS1: , lib:SOD-323_L1.8-W1.3-LS2.5-RD, F.Cu at (165.8, 95.5)
- added L1: , lib:IND-SMD_L4.0-W4.0, F.Cu at (161.5, 93.2)
- added R1: 62.5mW Thick Film Resistors 50V ±100ppm/℃ ±1% 14.3kΩ 0402 C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, lib:R0402, F.Cu at (163.1, 88.0)
- added R2: 62.5mW Thick Film Resistors 50V ±100ppm/℃ ±1% 4.3kΩ 0402 Ch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, lib:R0402, F.Cu at (161.1, 88.0)
- added U1: , lib:SOT-23-6_L2.9-W1.6-P0.95-LS2.8-BR, F.Cu at (166.0, 91.9)
Routing:
- net out: track 0.00 -> 8.33 mm, vias 0 -> 2
- net gnd: track 0.00 -> 7.10 mm, vias 0 -> 4
- net cb: track 0.00 -> 2.36 mm
- added copper zone on F.Cu, net sw
- added copper zone on F.Cu, net vcc
- added copper zone on F.Cu, net vcc-1
